File: groundslider.sch (KiCad schematic (older format))
At the start: 54 parts, among them P1 CONN_02X05, P2 CONN_02X05, P3 M3Drill, P4 M3Drill, P5 M3Drill, P6 M3Drill, P7 M3Drill, P8 CONN_01X05, P9 CONN_01X05, SW1 SPST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

Commit message: ハッチング前
Parts:
- P3, P4, P5, P6, P7: footprint hastech:M3_Drill -> kamiya:M3Drill2
Connections:
- net EZI2C_SCL: now also P9.4 (P4); no longer P9.3 (P3)
- net EZI2C_SDA: now also P9.3 (P3); no longer P9.4 (P4)
- net GND: now also P2.10 (P10); no longer P2.2 (P2), P3.1 (P1), P4.1 (P1), P5.1 (P1), P6.1 (P1), P7.1 (P1)
- net SPI_CS0: now also P2.3 (P3); no longer P2.7 (P7)
- net SPI_CS1: now also P2.4 (P4); no longer P2.8 (P8)
- net SPI_CS2: now also P2.1 (P1); no longer P2.9 (P9)
- net SPI_CS3: now also P2.2 (P2); no longer P2.10 (P10)
- net SPI_SCLK: now also P2.8 (P8); no longer P2.4 (P4)
- net VDD: now also P2.9 (P9); no longer P2.1 (P1)
- net XRES: now also P2.7 (P7); no longer P2.3 (P3)
- no-connect marks 14 -> 19
Changed lines of the file:
@@
 F 0 "P3" H 3200 6925 50  0000 C CNN
 F 1 "M3Drill" V 3300 6825 50  0000 C CNN
-F 2 "hastech:M3_Drill" H 3200 6825 50  0001 C CNN
+F 2 "kamiya:M3Drill2" H 3200 6825 50  0001 C CNN
 F 3 "" H 3200 6825 50  0000 C CNN
 	1    3200 6825
-	0    -1   -1   0
-$EndComp
-$Comp
-L CONN_01X01 P4
-U 1 1 56F786EA
-P 3500 6825
-F 0 "P4" H 3500 6925 50  0000 C CNN
-F 1 "M3Drill" V 3600 6825 50  0000 C CNN
-F 2 "hastech:M3_Drill" H 3500 6825 50  0001 C CNN
-F 3 "" H 3500 6825 50  0000 C CNN
-	1    3500 6825
 	0    -1   -1   0
 $EndComp
@@
 F 0 "P5" H 3800 6925 50  0000 C CNN
 F 1 "M3Drill" V 3900 6825 50  0000 C CNN
-F 2 "hastech:M3_Drill" H 3800 6825 50  0001 C CNN
+F 2 "kamiya:M3Drill2" H 3800 6825 50  0001 C CNN
 F 3 "" H 3800 6825 50  0000 C CNN
 	1    3800 6825
@@
 F 0 "P6" H 4100 6925 50  0000 C CNN
 F 1 "M3Drill" V 4200 6825 50  0000 C CNN
-F 2 "hastech:M3_Drill" H 4100 6825 50  0001 C CNN
+F 2 "kamiya:M3Drill2" H 4100 6825 50  0001 C CNN
 F 3 "" H 4100 6825 50  0000 C CNN
 	1    4100 6825
@@
 F 0 "P7" H 4375 6925 50  0000 C CNN
 F 1 "M3Drill" V 4475 6825 50  0000 C CNN
-F 2 "hastech:M3_Drill" H 4375 6825 50  0001 C CNN
+F 2 "kamiya:M3Drill2" H 4375 6825 50  0001 C CNN
 F 3 "" H 4375 6825 50  0000 C CNN
 	1    4375 6825
@@
 F 3 "" H 1625 5325 50  0000 C CNN
 	1    1625 6525
-	1    0    0    -1
+	1    0    0    1
 $EndComp
 $Comp
@@
 Text Label 2525 4150 1    60   ~ 0
 UART_TX
-Text Label 4975 6750 0    60   ~ 0
+Text Label 5000 6750 0    60   ~ 0
 UART_TX
 $Comp
@@
 	1    0    0    -1
 $EndComp
-$Comp
-L GND #PWR033
-U 1 1 56F8812D
-P 3200 7125
-F 0 "#PWR033" H 3200 6875 50  0001 C CNN
-F 1 "GND" H 3200 6975 50  0000 C CNN
-F 2 "" H 3200 7125 50  0000 C CNN
-F 3 "" H 3200 7125 50  0000 C CNN
-	1    3200 7125
-	1    0    0    -1
-$EndComp
 Wire Wire Line
 	3400 1250 3400 1200
@@
 	10775 4525 10775 4475
 Wire Wire Line
-	1375 5525 900  5525
+	900  5525 1375 5525
 Wire Wire Line
 	1375 5625 1025 5625
@@
 	5575 6650 5000 6650
 Wire Wire Line
-	5575 6750 4975 6750
+	5575 6750 5000 6750
 Wire Wire Line
 	2525 4150 2525 3775
@@
 Wire Wire Line
 	2625 1175 2625 1250
-Wire Wire Line
-	3200 7125 3200 7025
-Wire Wire Line
-	3200 7025 4375 7025
-Connection ~ 4100 7025
-Connection ~ 3800 7025
-Connection ~ 3500 7025
-Connection ~ 3200 7025
+Text Label 5000 6650 0    60   ~ 0
+EZI2C_SCL
 Text Label 5000 6550 0    60   ~ 0
-EZI2C_SCL
-Text Label 5000 6650 0    60   ~ 0
 EZI2C_SDA
 $Comp
@@
 Connection ~ 2625 4475
 Connection ~ 2625 4775
+$Comp
+L CONN_01X01 P4
+U 1 1 56F786EA
+P 3500 6825
+F 0 "P4" H 3500 6925 50  0000 C CNN
+F 1 "M3Drill" V 3600 6825 50  0000 C CNN
+F 2 "kamiya:M3Drill2" H 3500 6825 50  0001 C CNN
+F 3 "" H 3500 6825 50  0000 C CNN
+	1    3500 6825
+	0    -1   -1   0
+$EndComp
+NoConn ~ 4375 7025
+NoConn ~ 4100 7025
+NoConn ~ 3800 7025
+NoConn ~ 3500 7025
+NoConn ~ 3200 7025
 $EndSCHEMATC
