File: groundslider.kicad_pcb (KiCad board)
At the start: 2 copper layers, 54 parts, among them P1 CONN_02X05, P2 CONN_02X05, P3 M3Drill, P4 M3Drill, P5 M3Drill, P6 M3Drill, P7 M3Drill, P8 CONN_01X05, P9 CONN_01X05, SW1 SPST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

Commit message: CapSense配線
Parts:
- P1, R1, R10, R11, R12, R2, R3, R4, R5, R6, R7, R8, R9, U1: moved to B.Cu
- moved P3 165.6 mm to (60.0, 40.0)
- moved CS1 148.0 mm to (67.5, 55.0)
- moved R2 132.8 mm to (96.7, 110.3), turned to 315 degrees
- moved P4 129.7 mm to (60.0, 110.0)
- moved R5 127.6 mm to (100.4, 106.6), turned to 315 degrees
- moved CS2 126.9 mm to (67.5, 75.0)
- moved LED1 125.1 mm to (92.5, 120.0)
- moved LED0 123.2 mm to (67.5, 120.0)
- moved CS3 115.6 mm to (67.5, 95.0)
- moved R12 112.7 mm to (114.9, 112.3), turned to 225 degrees
- moved CS5 110.0 mm to (92.5, 75.0)
- moved R8 107.5 mm to (110.0, 107.4), turned to 225 degrees
- moved R6 102.2 mm to (99.1, 107.8), turned to 315 degrees
- moved R9 102.2 mm to (111.2, 108.6), turned to 225 degrees
- moved P1 101.6 mm to (55.0, 152.5), turned to 180 degrees
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Routing:
- net Net-(CS10-Pad1): track 0.00 -> 71.6 mm, vias 0 -> 1
- net Net-(CS1-Pad1): track 0.00 -> 70.8 mm, vias 0 -> 1
- net Net-(CS7-Pad1): track 0.00 -> 56.1 mm, vias 0 -> 1
- net Net-(CS4-Pad1): track 0.00 -> 55.2 mm, vias 0 -> 1
- net Net-(CS11-Pad1): track 0.00 -> 54.8 mm, vias 0 -> 1
- net Net-(CS2-Pad1): track 0.00 -> 54.6 mm, vias 0 -> 1
- net Net-(CS3-Pad1): track 0.00 -> 38.0 mm, vias 0 -> 1
- net Net-(CS12-Pad1): track 0.00 -> 37.9 mm, vias 0 -> 1
- net Net-(CS8-Pad1): track 0.00 -> 36.0 mm, vias 0 -> 1
- net Net-(CS5-Pad1): track 0.00 -> 35.8 mm, vias 0 -> 1
- net Net-(CS9-Pad1): track 0.00 -> 15.3 mm, vias 0 -> 1
- net Net-(CS6-Pad1): track 0.00 -> 14.7 mm, vias 0 -> 1
- net /CS20: track 0.00 -> 5.27 mm
- net /CS01: track 0.00 -> 5.04 mm
- net /CS23: track 0.00 -> 4.91 mm
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Other:
- board outline added: 100 x 100 mm
- net class CapSense added: clearance 0.2, trace_width 0.2032, via_dia 0.6, via_drill 0.4

Commit message: ハッチング前
Parts:
- C7, P2, P8, P9, R13: moved to B.Cu
- P3, P4, P5, P6, P7: footprint hastech:M3_Drill -> kamiya:M3Drill2
- moved SW3 147.1 mm to (81.9, 126.1), turned to 270 degrees
- moved C8 129.6 mm to (71.2, 123.9)
- moved C7 128.4 mm to (94.4, 118.6)
- moved SW2 128.3 mm to (83.6, 126.1), turned to 270 degrees
- moved C6 128.1 mm to (99.2, 119.9), turned to 180 degrees
- moved R13 127.1 mm to (97.4, 124.0), turned to 45 degrees
- moved C1 119.8 mm to (105.2, 122.0), turned to 180 degrees
- moved SW4 117.0 mm to (80.2, 126.1), turned to 270 degrees
- moved C2 111.3 mm to (105.1, 125.5), turned to 180 degrees
- moved C3 107.5 mm to (103.1, 117.8)
- moved C10 105.1 mm to (121.2, 123.7)
- moved SW1 104.9 mm to (85.3, 126.1), turned to 270 degrees
- moved C5 103.7 mm to (103.0, 119.9)
- moved C4 95.3 mm to (99.2, 117.8), turned to 180 degrees
- moved C11 88.3 mm to (146.2, 123.9)
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Connections:
- P2 pad 1: VDD -> /SPI_CS2
- P2 pad 10: /SPI_CS3 -> GND
- P2 pad 2: GND -> /SPI_CS3
- P2 pad 3: /XRES -> /SPI_CS0
- P2 pad 4: /SPI_SCLK -> /SPI_CS1
- P2 pad 7: /SPI_CS0 -> /XRES
- P2 pad 8: /SPI_CS1 -> /SPI_SCLK
- P2 pad 9: /SPI_CS2 -> VDD
- P9 pad 3: /EZI2C_SCL -> /EZI2C_SDA
- P9 pad 4: /EZI2C_SDA -> /EZI2C_SCL
Routing:
- net GND: track 0.00 -> 308.8 mm, vias 0 -> 33
- net VDD: track 0.00 -> 155.5 mm, vias 0 -> 5
- net /XRES: track 0.00 -> 111.2 mm, vias 0 -> 3
- net /SPI_SCLK: track 0.00 -> 108.0 mm, vias 0 -> 2
- net /SPI_MOSI: track 0.00 -> 106.4 mm, vias 0 -> 2
- net /SPI_CS3: track 0.00 -> 103.2 mm, vias 0 -> 1
- net /SPI_CS1: track 0.00 -> 100.8 mm, vias 0 -> 1
- net /SPI_MISO: track 0.00 -> 96.2 mm, vias 0 -> 2
- net /SPI_CS2: track 0.00 -> 95.9 mm, vias 0 -> 1
- net /SPI_CS0: track 0.00 -> 93.5 mm, vias 0 -> 1
- net /SWDIO: track 0.00 -> 29.1 mm, vias 0 -> 1
- net /SWDCK: track 0.00 -> 27.8 mm, vias 0 -> 1
- net Net-(LED1-Pad2): track 0.00 -> 24.9 mm
- net /SPI_CS: track 0.00 -> 21.5 mm, vias 0 -> 1
- net Net-(LED2-Pad2): track 0.00 -> 21.2 mm
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- added copper zone on B.Cu, net GND
- added copper zone on F.Cu, net GND
Other:
- net class Supply added: clearance 0.2, trace_width 0.3, via_dia 0.6, via_drill 0.4

Commit message: 表面ハッチング
Routing:
- net GND: track 308.8 -> 8777.4 mm, vias 33 -> 36
- net /LED_PWM: track 0.00 -> 44.3 mm, vias 0 -> 5

Commit message: 裏面ハッチング
Routing:
- net GND: track 8777.4 -> 14921.3 mm
- net Net-(CS5-Pad1): track 35.9 -> 40.7 mm
- net Net-(CS10-Pad1): track 76.4 -> 77.2 mm
